File: addon-edge-rpi-i2s-pmod.kicad_pcb (KiCad board)
At the start: 2 copper layers, 100 x 100 mm, 39 parts, among them J1 PMOD1, J10 Conn_01x02, J12 Conn_01x02, J13 Conn_01x01, J2 PMOD2, J3 PMOD3, J4 PMOD4, J5 Conn_01x06, J6 Conn_01x06, J7 Conn_01x03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

Commit message: generated gerber files
Routing:
- net /B14_SPI1_CE0_CLKBD: track 46.5 -> 50.2 mm
- net /B14_CE0_CLKBD: track 131.5 -> 134.2 mm
- net /B12_SRAMDQ12: track 104.2 -> 106.0 mm
- net /A1_MOSI: track 94.3 -> 95.9 mm
- net /A28_SPI1_MISO_WSBD: track 101.3 -> 102.7 mm
- net /SCL_RPI: track 45.7 -> 44.3 mm
- net /A1_SPI1_MOSI: track 81.6 -> 82.9 mm
- net /B11_SRAMDQ11: track 89.6 -> 90.9 mm
- net /B13_SCLK_DABD: track 124.0 -> 123.1 mm
- net /B13_SPI1_SCLK_DABD: track 52.3 -> 53.2 mm
- net +5V: track 158.8 -> 159.6 mm
- net /A27_DIN_I2S: track 115.7 -> 114.9 mm
- net /B3_SRAMDQ15: track 114.6 -> 115.3 mm
- net /A1_SPI0_MOSI: track 41.4 -> 42.1 mm
- net /A28_SPI0_MISO: track 32.8 -> 33.4 mm
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Other:
- board text added: "SPI0 (SPI SELECTION) SPI1"
- board text removed: "SPI0 / SPI1 SELECTION"

Commit message: v0.6 silkscreen and gerber updated
Parts:
- moved LO2 24.8 mm to (172.1, 114.3)
- moved LO1 3.17 mm to (167.7, 88.9)
- moved LO3 0.63 mm to (191.8, 61.6)
Other:
- board text added: "DAC POWER INPUT"
- board text added: "FOR MT32-PI SET JP4x SPI1, JP11 RPI, JUMPER ON JP12"
- board text added: "I2C OLED DISPLAY VERIFY 3V3/GND SOLDER JUMPERS JPS1, JPS2"
- board text added: "SOLDER CENTRAL PADS TO EITHER 3V3 OR GND"
- board text removed: "CHECK 3V3/GND SOLDER JUMPERS JPS1, JPS2"
- board text removed: "DAC VIN SOURCE"
- board text removed: "OLED DISPLAY"
Changed lines of the file:
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@@
     )
   )
-  (property "VERSION" "0.52")
+  (property "VERSION" "0.6")
   (net 0 "")
   (net 1 "/B26_WSEL_LRCLK_I2S")
@@
   (net 91 "/B27_SPI1CE2")
   (footprint "Symbol:OSHW-Logo2_9.8x8mm_SilkScreen" (layer "F.Cu")
-    (at 173.99 89.535)
+    (at 172.085 114.3)
     (descr "Open Source Hardware Symbol")
     (tags "Logo Symbol OSHW")
@@
   )
   (footprint "Symbol:KiCad-Logo2_12mm_SilkScreen" (layer "B.Cu")
-    (at 167.654893 92.112106 180)
+    (at 167.654893 88.937106 180)
     (descr "KiCad Logo")
     (tags "Logo KiCad")
@@
   )
   (footprint "Symbol:OSHW-Logo2_14.6x12mm_SilkScreen" (layer "B.Cu")
-    (at 191.77 60.96 180)
+    (at 191.77 61.595 180)
     (descr "Open Source Hardware Symbol")
     (tags "Logo Symbol OSHW")
@@
       ))
   )
+  (gr_rect (start 149.987 102.108) (end 169.418 108.458) (layer "B.SilkS") (width 0.12) (fill none))
+  (gr_line (start 133.985 77.7875) (end 133.35 77.1525) (layer "F.SilkS") (width 0.12))
+  (gr_rect (start 148.336 97.79) (end 168.402 104.14) (layer "F.SilkS") (width 0.12) (fill none))
+  (gr_line (start 132.08 77.7875) (end 133.985 77.7875) (layer "F.SilkS") (width 0.12))
   (gr_line (start 127 129.54) (end 126.365 128.905) (layer "F.SilkS") (width 0.12))
-  (gr_line (start 127 101.6) (end 127.635 102.235) (layer "F.SilkS") (width 0.12))
+  (gr_line (start 127 100.33) (end 127.635 100.965) (layer "F.SilkS") (width 0.12))
+  (gr_line (start 112.7125 77.7875) (end 110.8075 77.7875) (layer "F.SilkS") (width 0.12))
+  (gr_line (start 133.985 77.7875) (end 133.35 78.4225) (layer "F.SilkS") (width 0.12))
   (gr_circle (center 149.225 106.045) (end 150.7236 106.045) (layer "F.SilkS") (width 0.12) (fill solid))
-  (gr_line (start 127 103.505) (end 127 101.6) (layer "F.SilkS") (width 0.12))
-  (gr_line (start 127 101.6) (end 126.365 102.235) (layer "F.SilkS") (width 0.12))
+  (gr_rect (start 168.91 85.725) (end 183.515 93.98) (layer "F.SilkS") (width 0.12) (fill none))
+  (gr_line (start 127 102.235) (end 127 100.33) (layer "F.SilkS") (width 0.12))
+  (gr_line (start 127 100.33) (end 126.365 100.965) (layer "F.SilkS") (width 0.12))
   (gr_line (start 127 127.635) (end 127 129.54) (layer "F.SilkS") (width 0.12))
   (gr_line (start 127 129.54) (end 127.635 128.905) (layer "F.SilkS") (width 0.12))
+  (gr_line (start 110.8075 77.7875) (end 111.4425 77.1525) (layer "F.SilkS") (width 0.12))
+  (gr_line (start 110.8075 77.7875) (end 111.4425 78.4225) (layer "F.SilkS") (width 0.12))
   (gr_line (start 208.75 44.9397) (end 208.75 144.93875) (layer "Edge.Cuts") (width 0.05))
   (gr_line (start 140.335 44.9397) (end 208.75 44.9397) (layer "Edge.Cuts") (width 0.05))
@@
   (gr_line (start 108.75 144.93875) (end 108.75 72.9387) (layer "Edge.Cuts") (width 0.05))
   (gr_line (start 108.75 72.9387) (end 140.335 72.9387) (layer "Edge.Cuts") (width 0.05))
-  (gr_text "MIDI I2S SBC Pmod\nEdge Interface v${VERSION}\n\n" (at 167.64 114.3) (layer "B.SilkS")
+  (gr_text "MIDI I2S SBC Pmod\nEdge Interface v${VERSION}\n\n" (at 167.64 119.38) (layer "B.SilkS")
     (effects (font (size 1.5 1.5) (thickness 0.15)) (justify mirror))
   )
-  (gr_text "created by Hard Team Deca\nSomhic & Rhoderik & C.Palmero\n" (at 167.64 120.65) (layer "B.SilkS")
-    (effects (font (size 1.5 1.5) (thickness 0.15)) (justify mirror))
+  (gr_text "SOLDER CENTRAL PADS\nTO EITHER 3V3 OR GND" (at 168.783 105.283) (layer "B.SilkS")
+    (effects (font (size 1 1) (thickness 0.15)) (justify left mirror))
+  )
+  (gr_text "created by Hard Team Deca\nSomhic & Rhoderik & C.Palmero\n" (at 167.64 133.35) (layer "B.SilkS")
+    (effects (font (size 1 1) (thickness 0.15)) (justify mirror))
   )
   (gr_text "https://github.com/somhi/MIDI_I2S_SBC_Pmod_Edge_Interface" (at 167.64 137.795) (layer "B.SilkS")
@@
     (effects (font (size 0.75 0.75) (thickness 0.15)))
   )
-  (gr_text "OLED\nDISPLAY" (at 151.13 101.6) (layer "F.SilkS")
-    (effects (font (size 1.5 1.5) (thickness 0.15)) (justify left))
-  )
   (gr_text "3V3" (at 186.69 105.41) (layer "F.SilkS")
     (effects (font (size 1 1) (thickness 0.15)))
@@
     (effects (font (size 1 1) (thickness 0.15)))
   )
+  (gr_text "FOR MT32-PI SET \nJP4x SPI1,\nJP11 RPI, \nJUMPER ON JP12 " (at 176.53 90.17) (layer "F.SilkS")
+    (effects (font (size 1 1) (thickness 0.15)))
+  )
   (gr_text "BCLK" (at 116.205 86.36) (layer "F.SilkS")
     (effects (font (size 1 1) (thickness 0.15)) (justify left))
@@
     (effects (font (size 0.75 0.75) (thickness 0.15)))
   )
-  (gr_text "DAC VIN SOURCE" (at 154.305 60.96) (layer "F.SilkS")
+  (gr_text "DAC POWER INPUT" (at 154.305 60.325) (layer "F.SilkS")
     (effects (font (size 1 1) (thickness 0.15)))
   )
@@
     (effects (font (size 0.75 0.75) (thickness 0.15)))
   )
-  (gr_text "CHECK 3V3/GND\nSOLDER JUMPERS\nJPS1, JPS2" (at 140.97 111.125) (layer "F.SilkS")
+  (gr_text "I2C OLED DISPLAY\nVERIFY 3V3/GND SOLDER \nJUMPERS JPS1, JPS2" (at 148.844 100.965) (layer "F.SilkS")
     (effects (font (size 1 1) (thickness 0.15)) (justify left))
   )
@@
     (effects (font (size 0.75 0.75) (thickness 0.15)))
   )
-  (gr_text "SPI0 (SPI SELECTION) SPI1" (at 126.93 115.57 90) (layer "F.SilkS")
+  (gr_text "SPI0 (SPI SELECTION) SPI1" (at 126.93 114.935 90) (layer "F.SilkS")
     (effects (font (size 1 1) (thickness 0.15)))
   )
@@
     (effects (font (size 1 1) (thickness 0.15)))
   )
-  (gr_text "MIDI2SBC Edge v${VERSION}\n" (at 172.085 120.015) (layer "F.SilkS")
+  (gr_text "MIDI2SBC Edge v${VERSION}\n" (at 172.085 120.65) (layer "F.SilkS")
     (effects (font (size 1.5 1.5) (thickness 0.15)))
   )

Commit message: v0.7 sent to manufacturing
Other:
- board text added: "0.2000 mm / 0.2032 mm"
- board text added: "0.3000 mm"
- board text added: "1.6000 mm"
- board text added: "2"
- board text added: "99.9850 mm x 99.9990 mm"
- board text added: "BOARD CHARACTERISTICS"
- board text added: "Board Thickness:"
- board text added: "Board overall dimensions:"
- board text added: "Castellated pads:"
- board text added: "Copper Finish:"
- board text added: "Copper Layer Count:"
- board text added: "Edge card connectors:"
- board text added: "Impedance Control:"
- board text added: "Min hole diameter:"
- board text added: "Min track/spacing:"
- board text added: "No"
- board text added: "None"
- board text added: "Plated Board Edge:"
- board text added: "checklist: https://github.com/azonenberg/pcb-checklist/"
Changed lines of the file:
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@@
       (viasonmask false)
       (mode 1)
-      (useauxorigin true)
+      (useauxorigin false)
       (hpglpennumber 1)
       (hpglpenspeed 20)
@@
       (plotinvisibletext false)
       (sketchpadsonfab false)
-      (subtractmaskfromsilk false)
+      (subtractmaskfromsilk true)
       (outputformat 1)
       (mirror false)
@@
     )
   )
-  (property "VERSION" "0.6")
+  (property "VERSION" "0.7")
   (net 0 "")
   (net 1 "/B26_WSEL_LRCLK_I2S")
@@
   (gr_line (start 110.8075 77.7875) (end 111.4425 77.1525) (layer "F.SilkS") (width 0.12))
   (gr_line (start 110.8075 77.7875) (end 111.4425 78.4225) (layer "F.SilkS") (width 0.12))
-  (gr_line (start 208.75 44.9397) (end 208.75 144.93875) (layer "Edge.Cuts") (width 0.05))
-  (gr_line (start 140.335 44.9397) (end 208.75 44.9397) (layer "Edge.Cuts") (width 0.05))
-  (gr_line (start 108.75 144.93875) (end 208.75 144.93875) (layer "Edge.Cuts") (width 0.05))
-  (gr_line (start 140.335 72.9387) (end 140.335 44.9397) (layer "Edge.Cuts") (width 0.05))
-  (gr_line (start 108.75 144.93875) (end 108.75 72.9387) (layer "Edge.Cuts") (width 0.05))
-  (gr_line (start 108.75 72.9387) (end 140.335 72.9387) (layer "Edge.Cuts") (width 0.05))
+  (gr_line (start 208.725 44.9497) (end 208.725 144.93875) (layer "Edge.Cuts") (width 0.01))
+  (gr_line (start 140.335 44.9497) (end 208.725 44.9497) (layer "Edge.Cuts") (width 0.01))
+  (gr_line (start 108.75 144.93875) (end 208.725 144.93875) (layer "Edge.Cuts") (width 0.01))
+  (gr_line (start 140.335 72.9387) (end 140.335 44.9497) (layer "Edge.Cuts") (width 0.01))
+  (gr_line (start 108.75 144.93875) (end 108.75 72.9387) (layer "Edge.Cuts") (width 0.01))
+  (gr_line (start 108.75 72.9387) (end 140.335 72.9387) (layer "Edge.Cuts") (width 0.01))
   (gr_text "MIDI I2S SBC Pmod\nEdge Interface v${VERSION}\n\n" (at 167.64 119.38) (layer "B.SilkS")
     (effects (font (size 1.5 1.5) (thickness 0.15)) (justify mirror))
@@
     (effects (font (size 0.75 0.75) (thickness 0.15)))
   )
+  (gr_text "checklist: https://github.com/azonenberg/pcb-checklist/" (at 149.72 217.62) (layer "User.1")
+    (effects (font (size 3 3) (thickness 0.15)))
+  )
+  (gr_text "0.2000 mm / 0.2032 mm" (at 57.387143 44.98) (layer "User.1")
+    (effects (font (size 1.5 1.5) (thickness 0.2)) (justify left top))
+  )
+  (gr_text "Board Thickness: " (at 91.444286 35.95) (layer "User.1")
+    (effects (font (size 1.5 1.5) (thickness 0.2)) (justify left top))
+  )
+  (gr_text "Board overall dimensions: " (at 24.83 40.465) (layer "User.1")
+    (effects (font (size 1.5 1.5) (thickness 0.2)) (justify left top))
+  )
+  (gr_text "None" (at 57.387143 49.495) (layer "User.1")
+    (effects (font (size 1.5 1.5) (thickness 0.2)) (justify left top))
+  )
+  (gr_text "Castellated pads: " (at 24.83 54.01) (layer "User.1")
+    (effects (font (size 1.5 1.5) (thickness 0.2)) (justify left top))
+  )
+  (gr_text "Edge card connectors: " (at 24.83 58.525) (layer "User.1")
+    (effects (font (size 1.5 1.5) (thickness 0.2)) (justify left top))
+  )
+  (gr_text "No" (at 57.387143 58.525) (layer "User.1")
+    (effects (font (size 1.5 1.5) (thickness 0.2)) (justify left top))
+  )
+  (gr_text "0.3000 mm" (at 116.287143 44.98) (layer "User.1")
+    (effects (font (size 1.5 1.5) (thickness 0.2)) (justify left top))
+  )
+  (gr_text "99.9850 mm x 99.9990 mm" (at 57.387143 40.465) (layer "User.1")
+    (effects (font (size 1.5 1.5) (thickness 0.2)) (justify left top))
+  )
+  (gr_text "" (at 116.287143 40.465) (layer "User.1")
+    (effects (font (size 1.5 1.5) (thickness 0.2)) (justify left top))
+  )
+  (gr_text "Impedance Control: " (at 91.444286 49.495) (layer "User.1")
+    (effects (font (size 1.5 1.5) (thickness 0.2)) (justify left top))
+  )
+  (gr_text "No" (at 57.387143 54.01) (layer "User.1")
+    (effects (font (size 1.5 1.5) (thickness 0.2)) (justify left top))
+  )
+  (gr_text "Min hole diameter: " (at 91.444286 44.98) (layer "User.1")
+    (effects (font (size 1.5 1.5) (thickness 0.2)) (justify left top))
+  )
+  (gr_text "BOARD CHARACTERISTICS" (at 24.08 29.78) (layer "User.1")
+    (effects (font (size 2 2) (thickness 0.4)) (justify left top))
+  )
+  (gr_text "No" (at 116.287143 54.01) (layer "User.1")
+    (effects (font (size 1.5 1.5) (thickness 0.2)) (justify left top))
+  )
+  (gr_text "Min track/spacing: " (at 24.83 44.98) (layer "User.1")
+    (effects (font (size 1.5 1.5) (thickness 0.2)) (justify left top))
+  )
+  (gr_text "Plated Board Edge: " (at 91.444286 54.01) (layer "User.1")
+    (effects (font (size 1.5 1.5) (thickness 0.2)) (justify left top))
+  )
+  (gr_text "Copper Layer Count: " (at 24.83 35.95) (layer "User.1")
+    (effects (font (size 1.5 1.5) (thickness 0.2)) (justify left top))
+  )
+  (gr_text "No" (at 116.287143 49.495) (layer "User.1")
+    (effects (font (size 1.5 1.5) (thickness 0.2)) (justify left top))
+  )
+  (gr_text "2" (at 57.387143 35.95) (layer "User.1")
+    (effects (font (size 1.5 1.5) (thickness 0.2)) (justify left top))
+  )
+  (gr_text "1.6000 mm" (at 116.287143 35.95) (layer "User.1")
+    (effects (font (size 1.5 1.5) (thickness 0.2)) (justify left top))
+  )
+  (gr_text "Copper Finish: " (at 24.83 49.495) (layer "User.1")
+    (effects (font (size 1.5 1.5) (thickness 0.2)) (justify left top))
+  )
+  (gr_text "" (at 91.444286 40.465) (layer "User.1")
+    (effects (font (size 1.5 1.5) (thickness 0.2)) (justify left top))
+  )
   (dimension (type aligned) (layer "Dwgs.User")
-    (pts (xy 208.75 44.9397) (xy 208.75 144.93875))
+    (pts (xy 208.725 44.9497) (xy 208.725 144.93875))
     (height -10.96)
-    (gr_text "99.9990 mm" (at 217.805 94.615 90) (layer "Dwgs.User")
+    (gr_text "99.9891 mm" (at 217.805 94.615 90) (layer "Dwgs.User")
       (effects (font (size 1 1) (thickness 0.15)))
     )
@@
   )
   (dimension (type aligned) (layer "Dwgs.User")
-    (pts (xy 108.75 144.93875) (xy 208.75 144.93875))
+    (pts (xy 108.75 144.93875) (xy 208.725 144.93875))
     (height 9.36625)
-    (gr_text "100.0000 mm" (at 159.385 152.4) (layer "Dwgs.User")
+    (gr_text "99.9750 mm" (at 159.385 152.4) (layer "Dwgs.User")
       (effects (font (size 1 1) (thickness 0.15)))
     )
@@
     )
   )
+  (group "group-boardCharacteristics" (id 34b6b129-a76c-4a62-91cc-2743f5f4b2c4)
+    (members
+      4f0ad253-6758-4fab-a304-5619bb190326
+      5d6cfde2-9586-45a3-9d7e-b9db5ad7bc21
+      62cf0a26-9096-4000-923a-60daf3aa23f8
+      63777433-96ab-4b15-8870-c77f38cbb556
+      70e18146-fcad-491b-ae29-6b6b530cc027
+      738c73ca-416f-4cdc-b135-180d4d696484
+      7590e24b-577c-4fcd-9e1f-ab45b189df19
+      7cea007c-3280-4e58-94e8-fd0f1c985899
+      7f04153d-9d5e-47af-b99d-bc6a387c9a6f
+      897136b5-a5d5-4581-a6bf-48c25cde5ca5
+      8a80af2d-ce13-4b11-8a6d-9856813678bd
+      9b86d498-b713-4140-97c2-940c95f43f16
+      9fd2c636-f5cd-47e5-bbbc-56f7c25ff6b0
+      c7daa16d-2cdc-48f9-84e1-6fd3b9ab8609
+      d32ff0d3-6db2-4544-ab69-6c0b14790da2
+      ddcc8852-5683-4366-8128-1d6ff0a98b06
+      e0fafb5a-7612-49f2-857e-07a48cf36c67
+      e2eaff9d-4c94-4311-bec0-a13146b760ca
+      e34767e1-a29c-42c3-8abb-ef0a479b6adf
+      e66cdece-4893-4be4-8985-52fc83792731
+      e997c615-0a9d-46fc-872f-6b2d14f01b36
+      ed15d2ab-884d-4309-8fc5-a20c99e91302
+      f5156e03-6da9-4205-8d49-0997e01031c7
+    )
+  )
